File: pcb/kyutobodo_pcb.kicad_sch (KiCad schematic)
At the start: 298 parts, among them J1 OLED_128x64, SW1 SW_Push, SW10 SW_Push, SW11 SW_Push, SW12 SW_Push, SW13 SW_Push, SW14 SW_Push, SW15 SW_Push, SW16 SW_Push, SW17 SW_Push, SW18 SW_Push, SW19 SW_Push, SW2 SW_Push, SW20 SW_Push, SW21 SW_Push, SW22 SW_Push, SW23 SW_Push, SW24 SW_Push, SW25 SW_Push, SW26 SW_Push, SW27 SW_Push, SW28 SW_Push, SW29 SW_Push, SW3 SW_Push, SW30 SW_Push, SW31 SW_Push, SW32 SW_Push, SW33 SW_Push, SW34 SW_Push, SW35 SW_Push, SW36 SW_Push, SW37 SW_Push, SW38 SW_Push, SW39 SW_Push, SW4 SW_Push, SW40 SW_Push, SW41 SW_Push, SW42 SW_Push, SW43 SW_Push, SW44 SW_Push, SW45 SW_Push, SW46 SW_Push, SW47 SW_Push, SW48 SW_Push, SW49 SW_Push, SW5 SW_Push, SW50 SW_Push, SW51 SW_Push, SW52 SW_Push, SW53 SW_Push, SW54 SW_Push, SW55 SW_Push, SW56 SW_Push, SW57 SW_Push, SW58 SW_Push, SW59 SW_Push, SW6 SW_Push, SW60 SW_Push, SW61 SW_Push, SW62 SW_Push, SW63 SW_Push, SW64 SW_Push, SW65 SW_Push, SW66 SW_Push, SW67 SW_Push, SW68 SW_Push, SW69 SW_Push, SW7 SW_Push, SW70 RotaryEncoder_Switch, SW8 SW_Push, SW9 SW_Push, U1 Raspberry_Pi_Pico, U2 SN74LVC1T45DBV

Commit message: Schematic Revision 2
Parts:
- added JP1: SolderJumper_2_Bridged, KeebioParts:solder_jumper, symbol Jumper:SolderJumper_2_Bridged
- added R4, R5, R6, R7, R8: 10kΩ, symbol Device:R
- added R9: 470Ω, Resistor_SMD:R_0805_2012Metric_Pad1.20x1.40mm_HandSolder, symbol Device:R
- C2, C3: footprint Capacitor_SMD:C_0805_2012Metric_Pad1.18x1.45mm_HandSolder -> (none)
- D100, D101, D102, D103, D104, D105, D106, D107, D108, D109, D110, D111, D112, D113, D114, D115, D116, D117, D118, D119, D120, D121, D122, D123, D124, D125, D126, D127, D128, D129, D130, D131, D132, D133, D134, D135, D136, D137, D138, D139, D140, D141, D142, D143, D144, D70, D71, D72, D73, D74, D75, D76, D77, D78, D79, D80, D81, D82, D83, D84, D85, D86, D87, D88, D89, D90, D91, D92, D93, D94, D95, D96, D97, D98, D99: footprint LED_SMD:LED_SK6812MINI_PLCC4_3.5x3.5mm_P1.75mm -> KeebioParts:SK6812-MINI-E
- R1, R2: value 4.7kΩ -> 10kΩ; footprint ScottoKeebs_Hotswap:Hotswap_MX_1.00u -> (none)
- R3: value 470Ω -> 10kΩ; footprint ScottoKeebs_Hotswap:Hotswap_MX_1.00u -> (none)
Connections:
- net +3.3V: now also C2.1, R3.2, R4.2, R5.2, R6.2, R7.2, R8.2; no longer C3.2
- net +5V: now also C3.1; no longer C2.2
- net COL0: now also R1.1, SW17.1, SW2.1, SW32.1, SW46.1, SW61.1, U1.20 (GPIO15); no longer U1.21 (GPIO16)
- net COL1: now also R2.1, SW18.1, SW19.1, SW3.1, SW33.1, SW34.1, SW4.1, SW47.1, SW48.1, SW62.1, U1.19 (GPIO14); no longer SW17.1, SW2.1, SW32.1, SW46.1, SW61.1, U1.22 (GPIO17)
- net COL2: now also R3.1, SW20.1, SW21.1, SW35.1, SW36.1, SW49.1, SW5.1, SW50.1, SW6.1, U1.17 (GPIO13); no longer SW18.1, SW3.1, SW33.1, SW47.1, SW62.1, U1.24 (GPIO18)
- net COL3: now also SW22.1, SW23.1, SW37.1, SW38.1, SW51.1, SW52.1, SW63.1, SW7.1, SW8.1, U1.16 (GPIO12), R4.1; no longer SW19.1, SW34.1, SW4.1, SW48.1, U1.25 (GPIO19)
- net COL4: now also SW10.1, SW24.1, SW25.1, SW39.1, SW40.1, SW53.1, SW54.1, SW64.1, SW9.1, U1.15 (GPIO11), R5.1; no longer SW20.1, SW35.1, SW49.1, SW5.1, U1.26 (GPIO20)
- net COL5: now also SW11.1, SW12.1, SW26.1, SW27.1, SW41.1, SW42.1, SW55.1, SW56.1, SW65.1, SW66.1, U1.14 (GPIO10), R6.1; no longer SW21.1, SW36.1, SW50.1, SW6.1, U1.27 (GPIO21)
- net COL6: now also SW13.1, SW14.1, SW28.1, SW29.1, SW43.1, SW57.1, SW58.1, SW67.1, SW68.1, U1.12 (GPIO9), R7.1; no longer SW22.1, SW37.1, SW51.1, SW63.1, SW7.1, U1.29 (GPIO22)
- net COL7: now also SW15.1, SW30.1, SW44.1, SW59.1, SW69.1, U1.11 (GPIO8), R8.1; no longer SW23.1, SW38.1, SW52.1, SW8.1, U1.31 (GPIO26_ADC0)
- net EC11/SW: now also U1.2 (GPIO1); no longer U1.15 (GPIO11)
- net GND: now also C2.2, C3.2; no longer C2.1, C3.1
- net LED: now also JP1.1 (A)
- net ROW0: now also D10.2 (A), D12.2 (A), D14.2 (A), D2.2 (A), D4.2 (A), D6.2 (A), D8.2 (A), U1.21 (GPIO16); no longer D10.1 (K), D12.1 (K), D14.1 (K), D2.1 (K), D4.1 (K), D6.1 (K), D8.1 (K), U1.2 (GPIO1)
- net ROW1: now also D17.2 (A), D19.2 (A), D21.2 (A), D23.2 (A), D25.2 (A), D27.2 (A), D29.2 (A), U1.22 (GPIO17); no longer D17.1 (K), D19.1 (K), D21.1 (K), D23.1 (K), D25.1 (K), D27.1 (K), D29.1 (K), U1.9 (GPIO6)
- net ROW2: now also D32.2 (A), D34.2 (A), D36.2 (A), D38.2 (A), D40.2 (A), D42.2 (A), U1.24 (GPIO18); no longer D32.1 (K), D34.1 (K), D36.1 (K), D38.1 (K), D40.1 (K), D42.1 (K), U1.10 (GPIO7)
- net ROW3: now also D46.2 (A), D48.2 (A), D50.2 (A), D52.2 (A), D54.2 (A), D56.2 (A), D58.2 (A), U1.25 (GPIO19); no longer D46.1 (K), D48.1 (K), D50.1 (K), D52.1 (K), D54.1 (K), D56.1 (K), D58.1 (K), U1.11 (GPIO8)
- net ROW4: now also D61.2 (A), D64.2 (A), D66.2 (A), D68.2 (A), U1.26 (GPIO20); no longer D61.1 (K), D64.1 (K), D66.1 (K), D68.1 (K), U1.12 (GPIO9)
- net SSD1306/SCL: no longer R1.1
- net SSD1306/SDA: no longer R2.1
- net at SW14.2: now also D14.1 (K); no longer D14.2 (A)
- net at SW66.2: now also D66.1 (K); no longer D66.2 (A)
- net at SW6.2: now also D6.1 (K); no longer D6.2 (A)
- net at SW10.2: now also D10.1 (K); no longer D10.2 (A)
- net at SW42.2: now also D42.1 (K); no longer D42.2 (A)
- net at SW2.2: now also D2.1 (K); no longer D2.2 (A)
- net at SW38.2: now also D38.1 (K); no longer D38.2 (A)
- net at SW46.2: now also D46.1 (K); no longer D46.2 (A)
- net at SW54.2: now also D54.1 (K); no longer D54.2 (A)
- net at SW36.2: now also D36.1 (K); no longer D36.2 (A)
- net at SW29.2: now also D29.1 (K); no longer D29.2 (A)
- net at SW58.2: now also D58.1 (K); no longer D58.2 (A)
- net at SW56.2: now also D56.1 (K); no longer D56.2 (A)
- net at SW21.2: now also D21.1 (K); no longer D21.2 (A)
- net at SW23.2: now also D23.1 (K); no longer D23.2 (A)
- net at SW50.2: now also D50.1 (K); no longer D50.2 (A)
- net at SW27.2: now also D27.1 (K); no longer D27.2 (A)
- net at SW4.2: now also D4.1 (K); no longer D4.2 (A)
- net at SW52.2: now also D52.1 (K); no longer D52.2 (A)
- net at SW40.2: now also D40.1 (K); no longer D40.2 (A)
- net at U2.3 (A): now also JP1.2 (B), R9.1; no longer R3.1
- net at D70.3 (DIN): now also R9.2; no longer R3.2
- net at SW61.2: now also D61.1 (K); no longer D61.2 (A)
- net at SW8.2: now also D8.1 (K); no longer D8.2 (A)
- net at SW68.2: now also D68.1 (K); no longer D68.2 (A)
- net at SW48.2: now also D48.1 (K); no longer D48.2 (A)
- net at SW12.2: now also D12.1 (K); no longer D12.2 (A)
- net at SW19.2: now also D19.1 (K); no longer D19.2 (A)
- net at SW25.2: now also D25.1 (K); no longer D25.2 (A)
- net at SW32.2: now also D32.1 (K); no longer D32.2 (A)
- net at SW64.2: now also D64.1 (K); no longer D64.2 (A)
- net at SW17.2: now also D17.1 (K); no longer D17.2 (A)
- net at SW34.2: now also D34.1 (K); no longer D34.2 (A)
- removed net COL10: SW11.1, SW26.1, SW41.1, SW55.1, SW65.1, U1.20 (GPIO15)
- removed net COL11: SW12.1, SW27.1, SW42.1, SW56.1, SW66.1, U1.19 (GPIO14)
- removed net COL12: SW13.1, SW28.1, SW43.1, SW57.1, SW67.1, U1.17 (GPIO13)
- removed net COL13: SW14.1, SW29.1, SW58.1, SW68.1, U1.16 (GPIO12)
- removed net COL14: SW15.1, SW30.1, SW44.1, SW59.1, SW69.1, U1.14 (GPIO10)
- removed net COL8: SW24.1, SW39.1, SW53.1, SW9.1, U1.32 (GPIO27_ADC1)
- removed net COL9: SW10.1, SW25.1, SW40.1, SW54.1, SW64.1, U1.34 (GPIO28_ADC2)
- no-connect marks 8 -> 15
Other:
- note removed: "SWITCH MATRIX"
- moved on the sheet: D10, D12, D14, D17, D19, D2, D21, D23, D25, D27, D29, D32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

Commit message: Schematic Revision 3
Parts:
- removed R1, R2, R3, R4, R5, R6, R7, R8: 10kΩ, symbol Device:R
- C2, C3: footprint (none) -> Capacitor_SMD:C_0805_2012Metric_Pad1.18x1.45mm_HandSolder
- SW14: footprint ScottoKeebs_Hotswap:Hotswap_MX_1.00u -> ScottoKeebs_Hotswap:Hotswap_MX_2.00u
- SW16: footprint ScottoKeebs_Hotswap:Hotswap_MX_1.00u -> ScottoKeebs_Hotswap:Hotswap_MX_1.50u
- SW29: footprint ScottoKeebs_Hotswap:Hotswap_MX_1.00u -> ScottoKeebs_Hotswap:Hotswap_MX_ISOEnter
- SW31, SW67: footprint ScottoKeebs_Hotswap:Hotswap_MX_1.00u -> ScottoKeebs_Hotswap:Hotswap_MX_1.75u
- SW45, SW60, SW61, SW62: footprint ScottoKeebs_Hotswap:Hotswap_MX_1.00u -> ScottoKeebs_Hotswap:Hotswap_MX_1.25u
- SW63: footprint ScottoKeebs_Hotswap:Hotswap_MX_1.00u -> ScottoKeebs_Hotswap:Hotswap_MX_6.25u
- SW70: footprint ScottoKeebs_Scotto:Encoder_EC11_MX -> KeebioParts:RotaryEncoder_EC11
- U1: footprint Module:RaspberryPi_Pico_Common_THT -> ScottoKeebs_MCU:Raspberry_Pi_Pico
Connections:
- net COL0: now also U1.21 (GPIO16); no longer SW17.1, SW2.1, SW32.1, SW46.1, SW61.1, U1.20 (GPIO15)
- net COL1: now also SW17.1, SW2.1, SW32.1, SW46.1, SW61.1, U1.22 (GPIO17); no longer SW18.1, SW19.1, SW3.1, SW33.1, SW34.1, SW4.1, SW47.1, SW48.1, SW62.1, U1.19 (GPIO14)
- net COL2: now also SW18.1, SW3.1, SW33.1, SW47.1, SW62.1, U1.24 (GPIO18); no longer SW20.1, SW21.1, SW35.1, SW36.1, SW49.1, SW5.1, SW50.1, SW6.1, U1.17 (GPIO13)
- net COL3: now also SW19.1, SW34.1, SW4.1, SW48.1, U1.25 (GPIO19); no longer SW22.1, SW23.1, SW37.1, SW38.1, SW51.1, SW52.1, SW63.1, SW7.1, SW8.1, U1.16 (GPIO12)
- net COL4: now also SW20.1, SW35.1, SW49.1, SW5.1, U1.26 (GPIO20); no longer SW10.1, SW24.1, SW25.1, SW39.1, SW40.1, SW53.1, SW54.1, SW64.1, SW9.1, U1.15 (GPIO11)
- net COL5: now also SW21.1, SW36.1, SW50.1, SW6.1, U1.27 (GPIO21); no longer SW11.1, SW12.1, SW26.1, SW27.1, SW41.1, SW42.1, SW55.1, SW56.1, SW65.1, SW66.1, U1.14 (GPIO10)
- net COL6: now also SW22.1, SW37.1, SW51.1, SW63.1, SW7.1, U1.29 (GPIO22); no longer SW13.1, SW14.1, SW28.1, SW29.1, SW43.1, SW57.1, SW58.1, SW67.1, SW68.1, U1.12 (GPIO9)
- net COL7: now also SW23.1, SW38.1, SW52.1, SW8.1, U1.31 (GPIO26_ADC0); no longer SW15.1, SW30.1, SW44.1, SW59.1, SW69.1, U1.11 (GPIO8)
- net ROW0: now also D10.1 (K), D12.1 (K), D14.1 (K), D2.1 (K), D4.1 (K), D6.1 (K), D8.1 (K), U1.20 (GPIO15); no longer D10.2 (A), D12.2 (A), D14.2 (A), D2.2 (A), D4.2 (A), D6.2 (A), D8.2 (A), U1.21 (GPIO16)
- net ROW1: now also D17.1 (K), D19.1 (K), D21.1 (K), D23.1 (K), D25.1 (K), D27.1 (K), D29.1 (K), U1.19 (GPIO14); no longer D17.2 (A), D19.2 (A), D21.2 (A), D23.2 (A), D25.2 (A), D27.2 (A), D29.2 (A), U1.22 (GPIO17)
- net ROW2: now also D32.1 (K), D34.1 (K), D36.1 (K), D38.1 (K), D40.1 (K), D42.1 (K), U1.17 (GPIO13); no longer D32.2 (A), D34.2 (A), D36.2 (A), D38.2 (A), D40.2 (A), D42.2 (A), U1.24 (GPIO18)
- net ROW3: now also D46.1 (K), D48.1 (K), D50.1 (K), D52.1 (K), D54.1 (K), D56.1 (K), D58.1 (K), U1.16 (GPIO12); no longer D46.2 (A), D48.2 (A), D50.2 (A), D52.2 (A), D54.2 (A), D56.2 (A), D58.2 (A), U1.25 (GPIO19)
- net ROW4: now also D61.1 (K), D64.1 (K), D66.1 (K), D68.1 (K), U1.15 (GPIO11); no longer D61.2 (A), D64.2 (A), D66.2 (A), D68.2 (A), U1.26 (GPIO20)
- net at SW14.2: now also D14.2 (A); no longer D14.1 (K)
- net at SW66.2: now also D66.2 (A); no longer D66.1 (K)
- net at SW6.2: now also D6.2 (A); no longer D6.1 (K)
- net at SW10.2: now also D10.2 (A); no longer D10.1 (K)
- net at SW42.2: now also D42.2 (A); no longer D42.1 (K)
- net at SW2.2: now also D2.2 (A); no longer D2.1 (K)
- net at SW38.2: now also D38.2 (A); no longer D38.1 (K)
- net at SW46.2: now also D46.2 (A); no longer D46.1 (K)
- net at SW54.2: now also D54.2 (A); no longer D54.1 (K)
- net at SW36.2: now also D36.2 (A); no longer D36.1 (K)
- net at SW29.2: now also D29.2 (A); no longer D29.1 (K)
- net at SW58.2: now also D58.2 (A); no longer D58.1 (K)
- net at SW56.2: now also D56.2 (A); no longer D56.1 (K)
- net at SW21.2: now also D21.2 (A); no longer D21.1 (K)
- net at SW23.2: now also D23.2 (A); no longer D23.1 (K)
- net at SW50.2: now also D50.2 (A); no longer D50.1 (K)
- net at SW27.2: now also D27.2 (A); no longer D27.1 (K)
- net at SW4.2: now also D4.2 (A); no longer D4.1 (K)
- net at SW52.2: now also D52.2 (A); no longer D52.1 (K)
- net at SW40.2: now also D40.2 (A); no longer D40.1 (K)
- net at SW61.2: now also D61.2 (A); no longer D61.1 (K)
- net at SW8.2: now also D8.2 (A); no longer D8.1 (K)
- net at SW68.2: now also D68.2 (A); no longer D68.1 (K)
- net at SW48.2: now also D48.2 (A); no longer D48.1 (K)
- net at SW12.2: now also D12.2 (A); no longer D12.1 (K)
- net at SW19.2: now also D19.2 (A); no longer D19.1 (K)
- net at SW25.2: now also D25.2 (A); no longer D25.1 (K)
- net at SW32.2: now also D32.2 (A); no longer D32.1 (K)
- net at SW64.2: now also D64.2 (A); no longer D64.1 (K)
- net at SW17.2: now also D17.2 (A); no longer D17.1 (K)
- net at SW34.2: now also D34.2 (A); no longer D34.1 (K)
- net COL13: now reaches U1.10 (GPIO7)
- net COL13: now also SW14.1, SW29.1, SW58.1, SW68.1
- net COL8: now reaches U1.32 (GPIO27_ADC1)
- net COL8: now also SW24.1, SW39.1, SW53.1, SW9.1
- net COL9: now reaches U1.34 (GPIO28_ADC2)
- net COL9: now also SW10.1, SW25.1, SW40.1, SW54.1, SW64.1
- net COL14: now reaches U1.9 (GPIO6)
- net COL14: now also SW15.1, SW30.1, SW44.1, SW59.1, SW69.1
- new net COL10: SW11.1, SW26.1, SW41.1, SW55.1, SW65.1, U1.14 (GPIO10)
- new net COL11: SW12.1, SW27.1, SW42.1, SW56.1, SW66.1, U1.12 (GPIO9)
- new net COL12: SW13.1, SW28.1, SW43.1, SW57.1, SW67.1, U1.11 (GPIO8)
- no-connect marks 15 -> 8
Other:
- moved on the sheet: D10, D12, D14, D17, D19, D2, D21, D23, D25, D27, D29, D32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

Commit message: Schematic Revision 4
Parts:
- removed C78: 0.1uF, Capacitor_SMD:C_0805_2012Metric_Pad1.18x1.45mm_HandSolder, symbol Device:C_Small
- removed D144: SK6812MINI-E, KeebioParts:SK6812-MINI-E, symbol LED:SK6812MINI
- SW57: footprint ScottoKeebs_Hotswap:Hotswap_MX_1.00u -> ScottoKeebs_Hotswap:Hotswap_MX_1.75u
- SW67: footprint ScottoKeebs_Hotswap:Hotswap_MX_1.75u -> ScottoKeebs_Hotswap:Hotswap_MX_1.00u
